Commit message: changed mesh locations

File: turtlebot3_gazebo/urdf/turtlebot3_burger.urdf (robot description, URDF)
Before this commit: robot turtlebot3_burger, 7 links, 6 joints
Links:
- removed link base_scan
- added link velodyne, mass 0.114; collision cylinder length=0.0315 radius=0.055; visual mesh filename=package://velodyne_description/meshes/VLP16_scan.dae scale=0.001 0.001 0.001
Joints:
- joint scan_joint: child base_scan -> velodyne

Commit message: added ground truth and base scan to burger model

File: turtlebot3_gazebo/urdf/turtlebot3_burger.urdf (robot description, URDF)
Before this commit: robot turtlebot3_burger, 7 links, 6 joints
Links:
- added link base_scan, mass 0.114; collision cylinder length=0.0315 radius=0.055; visual mesh filename=package://turtlebot3_gazebo/models/turtlebot3_common/meshes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 scale=0.001 0.001 0.001
Joints:
- added joint velodyne_joint: type fixed, parent base_link, child velodyne, origin xyz=-0.032 0 0.172 rpy=0 0 0
- joint scan_joint: child velodyne -> base_scan
